Commit message: fix(urdf): 更新四足机器人URDF模型的连杆和关节配置
替换原有STL网格为基础几何形状，调整关节限位范围与连杆姿态，修正关节轴方向参数

File: unitree_model/geesun_dog/geesun-dog/dog1/urdf/dog1.urdf (robot description, URDF)
Before this commit: robot dog1, 13 links, 12 joints
Links:
- link Link_fl_hip: geometry collision cylinder length=0.09 radius=0.05; collision cylinder length=0.25 radius=0.05
- link Link_fr_hip: geometry collision cylinder length=0.09 radius=0.05; collision cylinder length=0.25 radius=0.05
- link Link_hl_hip: geometry collision cylinder length=0.09 radius=0.05; collision cylinder length=0.25 radius=0.05
- link Link_hr_hip: geometry collision cylinder length=0.09 radius=0.05; collision cylinder length=0.25 radius=0.05
Joints:
- joint joint_fl_calf: axis 0 -1 0 -> 0 1 0; limit lower=0 upper=0 effort=0 velocity=0 -> lower=-0.19198621771937624 upper=1.6929693744344996 effort=0 velocity=0
- joint joint_fl_hip: limit lower=0 upper=0 effort=0 velocity=0 -> lower=-1.0471975511965976 upper=1.0471975511965976 effort=0 velocity=0
- joint joint_fl_thigh: axis 0 -1 0 -> 0 1 0; limit lower=0 upper=0 effort=0 velocity=0 -> lower=-1.3439035240356338 upper=3.717551306747922 effort=0 velocity=0
- joint joint_fr_calf: axis 0 0.99947 0.032517 -> 0 1 0; limit lower=0 upper=0 effort=0 velocity=0 -> lower=-0.8377580409572781 upper=1.0471975511965976 effort=0 velocity=0
- joint joint_fr_hip: limit lower=0 upper=0 effort=0 velocity=0 -> lower=-1.0471975511965976 upper=1.0471975511965976 effort=0 velocity=0
- joint joint_fr_thigh: axis 0 0.99947 0.032517 -> 0 1 0; limit lower=0 upper=0 effort=0 velocity=0 -> lower=-1.57 upper=3.49 effort=0 velocity=0
- joint joint_hl_calf: axis 0 -1 0 -> 0 1 0; limit lower=0 upper=0 effort=0 velocity=0 -> lower=-0.13962634015954636 upper=1.7453292519943295 effort=0 velocity=0
- joint joint_hl_hip: axis -1 0 0 -> 1 0 0; limit lower=0 upper=0 effort=0 velocity=0 -> lower=-1.0471975511965976 upper=1.0471975511965976 effort=0 velocity=0
- joint joint_hl_thigh: axis 0 -1 0 -> 0 1 0; limit lower=0 upper=0 effort=0 velocity=0 -> lower=-0.7504915783575616 upper=4.310963252425994 effort=0 velocity=0
- joint joint_hr_calf: limit lower=0 upper=0 effort=0 velocity=0 -> lower=0.20943951023931953 upper=2.0943951023931953 effort=0 velocity=0
- joint joint_hr_hip: axis -1 0 0 -> 1 0 0; limit lower=0 upper=0 effort=0 velocity=0 -> lower=-1.0471975511965976 upper=1.0471975511965976 effort=0 velocity=0
- joint joint_hr_thigh: limit lower=0 upper=0 effort=0 velocity=0 -> lower=-0.7853981633974483 upper=4.276056667386107 effort=0 velocity=0
