Commit message: docs: 更新四足机器人URDF模型及关联网格文件
替换原有URDF模型文件，更新机器人命名、连杆关节结构、惯性参数及碰撞几何
删除旧的STL网格文件，使用SolidWorks导出的新URDF配置

File: geesun_dog_urdf/geesun-dog/lingsi_d30w/urdf/lingsi_d30w.urdf (robot description, URDF)
Before this commit: robot lingsi_d30w, 17 links, 16 joints
Links:
- removed link base_link
- removed link link_fl_calf
- removed link link_fl_hip
- removed link link_fl_thigh
- removed link link_fl_wheel
- removed link link_fr_calf
- removed link link_fr_hip
- removed link link_fr_thigh
- removed link link_fr_wheel
- removed link link_hl_calf
- removed link link_hl_hip
- removed link link_hl_thigh
- removed link link_hl_wheel
- removed link link_hr_calf
- removed link link_hr_hip
- removed link link_hr_thigh
- removed link link_hr_wheel
- added link FL_calf, mass 1.04303800302805; collision box size=0.01 0.026 0.056; collision box size=0.01 0.026 0.08
- added link FL_hip, mass 1.655; collision cylinder length=0.175 radius=0.0625; visual mesh filename=../meshes/FL_hip.STL
- added link FL_thigh, mass 2.085; collision box size=0.07 0.04 0.28; visual mesh filename=../meshes/FL_thigh.STL
- added link FL_wheel, mass 0.998507; collision cylinder length=0.008 radius=0.09328; collision cylinder length=0.008 radius=0.09328
- added link FR_calf, mass 1.04301180606178; collision box size=0.01 0.026 0.056; collision box size=0.01 0.026 0.08
- added link FR_hip, mass 1.655; collision cylinder length=0.175 radius=0.0625; visual mesh filename=../meshes/FR_hip.STL
- added link FR_thigh, mass 2.085; collision box size=0.07 0.04 0.28; visual mesh filename=../meshes/FR_thigh.STL
- added link FR_wheel, mass 0.998507; collision cylinder length=0.008 radius=0.09328; collision cylinder length=0.008 radius=0.09328
- added link RL_calf, mass 1.04303800470918; collision box size=0.01 0.026 0.056; collision box size=0.01 0.026 0.08
- added link RL_hip, mass 1.655; collision cylinder length=0.175 radius=0.0625; visual mesh filename=../meshes/RL_hip.STL
- added link RL_thigh, mass 2.085; collision box size=0.07 0.04 0.28; visual mesh filename=../meshes/RL_thigh.STL
- added link RL_wheel, mass 0.998507; collision cylinder length=0.008 radius=0.09328; collision cylinder length=0.008 radius=0.09328
- added link RR_calf, mass 1.04301180268041; collision box size=0.01 0.026 0.056; collision box size=0.01 0.026 0.08
- added link RR_hip, mass 1.655; collision cylinder length=0.175 radius=0.0625; visual mesh filename=../meshes/RR_hip.STL
- added link RR_thigh, mass 2.085; collision box size=0.07 0.04 0.28; visual mesh filename=../meshes/RR_thigh.STL
- added link RR_wheel, mass 0.998507; collision cylinder length=0.008 radius=0.09328; collision cylinder length=0.008 radius=0.09328
- added link trunk, mass 17.360; collision box size=1.0 0.26 0.22; visual mesh filename=../meshes/base_link.STL
Joints:
- removed joint joint_fl_calf
- removed joint joint_fl_hip
- removed joint joint_fl_thigh
- removed joint joint_fl_wheel
- removed joint joint_fr_calf
- removed joint joint_fr_hip
- removed joint joint_fr_thigh
- removed joint joint_fr_wheel
- removed joint joint_hl_calf
- removed joint joint_hl_hip
- removed joint joint_hl_thigh
- removed joint joint_hl_wheel
- removed joint joint_hr_calf
- removed joint joint_hr_hip
- removed joint joint_hr_thigh
- removed joint joint_hr_wheel
- added joint FL_calf_joint: type revolute, parent FL_thigh, child FL_calf, origin xyz=0 0 -0.28 rpy=0 0 0, axis 0 -1 0, limit lower=0.536 upper=2.775 effort=160.0 velocity=15.0
- added joint FL_hip_joint: type revolute, parent trunk, child FL_hip, origin xyz=0.2755 0.085 0 rpy=0 0 0, axis 1 0 0, limit lower=-0.698 upper=0.698 effort=100.0 velocity=20.0
- added joint FL_thigh_joint: type revolute, parent FL_hip, child FL_thigh, origin xyz=0 0.0905 0 rpy=0 0 0, axis 0 -1 0, limit lower=-3.054 upper=1.0 effort=100.0 velocity=20.0
- added joint FL_wheel_motor: type revolute, parent FL_calf, child FL_wheel, origin xyz=0 0.0676 -0.275 rpy=0 0 0, axis 0 -1 0, limit lower=-999999 upper=999999 effort=14.0 velocity=65
- added joint FR_calf_joint: type revolute, parent FR_thigh, child FR_calf, origin xyz=0 0 -0.28 rpy=0 0 0, axis 0 -1 0, limit lower=0.536 upper=2.775 effort=160.0 velocity=15.0
- added joint FR_hip_joint: type revolute, parent trunk, child FR_hip, origin xyz=0.2755 -0.085 0 rpy=0 0 0, axis 1 0 0, limit lower=-0.698 upper=0.698 effort=100.0 velocity=20.0
- added joint FR_thigh_joint: type revolute, parent FR_hip, child FR_thigh, origin xyz=0 -0.0905 0 rpy=0 0 0, axis 0 -1 0, limit lower=-3.054 upper=1.0 effort=100.0 velocity=20.0
- added joint FR_wheel_motor: type revolute, parent FR_calf, child FR_wheel, origin xyz=0 -0.0676 -0.275 rpy=0 0 0, axis 0 -1 0, limit lower=-999999 upper=999999 effort=14.0 velocity=65
- added joint RL_calf_joint: type revolute, parent RL_thigh, child RL_calf, origin xyz=0 0 -0.28 rpy=0 0 0, axis 0 -1 0, limit lower=0.536 upper=2.775 effort=160.0 velocity=15.0
- added joint RL_hip_joint: type revolute, parent trunk, child RL_hip, origin xyz=-0.2755 0.085 0 rpy=0 0 0, axis 1 0 0, limit lower=-0.698 upper=0.698 effort=100.0 velocity=20.0
- added joint RL_thigh_joint: type revolute, parent RL_hip, child RL_thigh, origin xyz=0 0.0905 0 rpy=0 0 0, axis 0 -1 0, limit lower=-3.054 upper=1.0 effort=100.0 velocity=20.0
- added joint RL_wheel_motor: type revolute, parent RL_calf, child RL_wheel, origin xyz=0 0.0676 -0.275 rpy=0 0 0, axis 0 -1 0, limit lower=-999999 upper=999999 effort=14.0 velocity=65
- added joint RR_calf_joint: type revolute, parent RR_thigh, child RR_calf, origin xyz=0 0 -0.28 rpy=0 0 0, axis 0 -1 0, limit lower=0.536 upper=2.775 effort=160.0 velocity=15.0
- added joint RR_hip_joint: type revolute, parent trunk, child RR_hip, origin xyz=-0.2755 -0.085 0 rpy=0 0 0, axis 1 0 0, limit lower=-0.698 upper=0.698 effort=100.0 velocity=20.0
- added joint RR_thigh_joint: type revolute, parent RR_hip, child RR_thigh, origin xyz=0 -0.0905 0 rpy=0 0 0, axis 0 -1 0, limit lower=-3.054 upper=1.0 effort=100.0 velocity=20.0
- added joint RR_wheel_motor: type revolute, parent RR_calf, child RR_wheel, origin xyz=0 -0.0676 -0.275 rpy=0 0 0, axis 0 -1 0, limit lower=-999999 upper=999999 effort=14.0 velocity=65

Commit message: docs: 添加四足机器人A01mw的URDF模型及相关文档

File: geesun_dog_urdf/geesun-dog/lingsi_d30w/urdf/lingsi_d30w.urdf (robot description, URDF)
Before this commit: robot A01mW, 17 links, 16 joints
Links:
- removed link FL_wheel
- removed link FR_wheel
- removed link RL_wheel
- removed link RR_wheel
- removed link trunk
- added link base_inertia, mass 17.360
- added link base_link; collision mesh filename=package://quad_description/meshes/A01mw/base_link.STL; visual mesh filename=package://quad_description/meshes/A01mw/base_link.STL
- added link fl_wheel, mass 0.99851; collision mesh filename=package://quad_description/meshes/A01mw/FL_wheel.STL; visual mesh filename=package://quad_description/meshes/A01mw/FL_wheel.STL
- added link fr_wheel, mass 0.9985; collision mesh filename=package://quad_description/meshes/A01mw/FR_wheel.STL; visual mesh filename=package://quad_description/meshes/A01mw/FR_wheel.STL
- added link hl_wheel, mass 0.85845; collision mesh filename=package://quad_description/meshes/A01mw/RL_wheel.STL; visual mesh filename=package://quad_description/meshes/A01mw/RL_wheel.STL
- added link hr_wheel, mass 0.85845; collision mesh filename=package://quad_description/meshes/A01mw/RR_wheel.STL; visual mesh filename=package://quad_description/meshes/A01mw/RR_wheel.STL
- link FL_calf: geometry collision mesh filename=package://quad_description/meshes/A01mw/FL_calf.STL; visual mesh filename=package://quad_description/meshes/A01mw/FL_calf.STL
- link FL_hip: geometry collision mesh filename=package://quad_description/meshes/A01mw/FL_hip.STL; visual mesh filename=package://quad_description/meshes/A01mw/FL_hip.STL
- link FL_thigh: geometry collision mesh filename=package://quad_description/meshes/A01mw/FL_thigh.STL; visual mesh filename=package://quad_description/meshes/A01mw/FL_thigh.STL
- link FR_calf: geometry collision mesh filename=package://quad_description/meshes/A01mw/FR_calf.STL; visual mesh filename=package://quad_description/meshes/A01mw/FR_calf.STL
- link FR_hip: geometry collision mesh filename=package://quad_description/meshes/A01mw/FR_hip.STL; visual mesh filename=package://quad_description/meshes/A01mw/FR_hip.STL
- link FR_thigh: geometry collision mesh filename=package://quad_description/meshes/A01mw/FR_thigh.STL; visual mesh filename=package://quad_description/meshes/A01mw/FR_thigh.STL
- link RL_calf: mass 1.04303800470918 -> 1.04301180268041; geometry collision mesh filename=package://quad_description/meshes/A01mw/RL_calf.STL; visual mesh filename=package://quad_description/meshes/A01mw/RL_calf.STL
- link RL_hip: geometry collision mesh filename=package://quad_description/meshes/A01mw/RL_hip.STL; visual mesh filename=package://quad_description/meshes/A01mw/RL_hip.STL
- link RL_thigh: geometry collision mesh filename=package://quad_description/meshes/A01mw/RL_thigh.STL; visual mesh filename=package://quad_description/meshes/A01mw/RL_thigh.STL
- link RR_calf: mass 1.04301180268041 -> 1.04303800470918; geometry collision mesh filename=package://quad_description/meshes/A01mw/RR_calf.STL; visual mesh filename=package://quad_description/meshes/A01mw/RR_calf.STL
- link RR_hip: geometry collision mesh filename=package://quad_description/meshes/A01mw/RR_hip.STL; visual mesh filename=package://quad_description/meshes/A01mw/RR_hip.STL
- link RR_thigh: geometry collision mesh filename=package://quad_description/meshes/A01mw/RR_thigh.STL; visual mesh filename=package://quad_description/meshes/A01mw/RR_thigh.STL
Joints:
- removed joint FL_calf_joint
- removed joint FL_hip_joint
- removed joint FL_thigh_joint
- removed joint FL_wheel_motor
- removed joint FR_calf_joint
- removed joint FR_hip_joint
- removed joint FR_thigh_joint
- removed joint FR_wheel_motor
- removed joint RL_calf_joint
- removed joint RL_hip_joint
- removed joint RL_thigh_joint
- removed joint RL_wheel_motor
- removed joint RR_calf_joint
- removed joint RR_hip_joint
- removed joint RR_thigh_joint
- removed joint RR_wheel_motor
- added joint base_inertia_to_base: type fixed, parent base_link, child base_inertia, origin xyz=0 0 0 rpy=0 0 0
- added joint fl_wheel_joint: type revolute, parent FL_calf, child fl_wheel, origin xyz=0 0.0676 -0.27498 rpy=0 0 0, axis 0 1 0, limit lower=-999999 upper=999999 effort=20.0 velocity=65
- added joint fr_wheel_joint: type revolute, parent FR_calf, child fr_wheel, origin xyz=0 -0.0676 -0.275 rpy=0 0 0, axis 0 -1 0, limit lower=-999999 upper=999999 effort=20.0 velocity=65
- added joint hl_wheel_joint: type revolute, parent RL_calf, child hl_wheel, origin xyz=0 0.0676 -0.275 rpy=0 0 0, axis 0 -1 0, limit lower=-999999 upper=999999 effort=20.0 velocity=65
- added joint hr_wheel_joint: type revolute, parent RR_calf, child hr_wheel, origin xyz=0 -0.0676 -0.27498 rpy=0 0 0, axis 0 -1 0, limit lower=-999999 upper=999999 effort=20.0 velocity=65
- added joint leg0_fr_joint0: type revolute, parent base_link, child FR_hip, origin xyz=0.2755 -0.085 0 rpy=0 0 0, axis 1 0 0, limit lower=-0.6981 upper=0.6981 effort=72 velocity=27
- added joint leg0_fr_joint1: type revolute, parent FR_hip, child FR_thigh, origin xyz=0 -0.0905 0 rpy=0 0 0, axis 0 -1 0, limit lower=-3.05 upper=0.6981 effort=72 velocity=27
- added joint leg0_fr_joint2: type revolute, parent FR_thigh, child FR_calf, origin xyz=0 0 -0.28 rpy=0 0 0, axis 0 -1 0, limit lower=0.525 upper=2.765 effort=136 velocity=14
- added joint leg1_fl_joint0: type revolute, parent base_link, child FL_hip, origin xyz=0.2755 0.085 0 rpy=0 0 0, axis 1 0 0, limit lower=-0.6981 upper=0.6981 effort=72 velocity=27
- added joint leg1_fl_joint1: type revolute, parent FL_hip, child FL_thigh, origin xyz=0 0.0905 0 rpy=0 0 0, axis 0 -1 0, limit lower=-3.05 upper=0.6981 effort=72 velocity=27
- added joint leg1_fl_joint2: type revolute, parent FL_thigh, child FL_calf, origin xyz=0 0 -0.28 rpy=0 0 0, axis 0 -1 0, limit lower=0.525 upper=2.765 effort=136 velocity=14
- added joint leg2_hr_joint0: type revolute, parent base_link, child RR_hip, origin xyz=-0.2755 -0.085 0 rpy=0 0 0, axis 1 0 0, limit lower=-0.6981 upper=0.6981 effort=72 velocity=27
- added joint leg2_hr_joint1: type revolute, parent RR_hip, child RR_thigh, origin xyz=0 -0.0905 0 rpy=0 0 0, axis 0 -1 0, limit lower=-3.05 upper=0.6981 effort=72 velocity=27
- added joint leg2_hr_joint2: type revolute, parent RR_thigh, child RR_calf, origin xyz=0 0 -0.28 rpy=0 0 0, axis 0 -1 0, limit lower=0.525 upper=2.765 effort=136 velocity=14
- added joint leg3_hl_joint0: type revolute, parent base_link, child RL_hip, origin xyz=-0.2755 0.085 0 rpy=0 0 0, axis 1 0 0, limit lower=-0.698 upper=0.698 effort=100.0 velocity=20.0
- added joint leg3_hl_joint1: type revolute, parent RL_hip, child RL_thigh, origin xyz=0 0.0905 0 rpy=0 0 0, axis 0 -1 0, limit lower=-3.05 upper=0.6981 effort=72 velocity=27
- added joint leg3_hl_joint2: type revolute, parent RL_thigh, child RL_calf, origin xyz=0 0 -0.28 rpy=0 0 0, axis 0 -1 0, limit lower=0.525 upper=2.765 effort=136 velocity=14
